Commit message: Add Lite3 description package and files

File: Lite3_description/Lite3/urdf/Lite3.urdf (robot description, URDF)
Before this commit: robot MiniLiteV3, 18 links, 17 joints
Links:
- added link front_link; visual box size=0.2 0.2 0.02
- added link rear_link; visual box size=0.2 0.2 0.02
Joints:
- added joint front_joint: type fixed, parent TORSO, child front_link, origin xyz=0 0 0.1 rpy=0 0 0
- added joint rear_joint: type fixed, parent TORSO, child rear_link, origin xyz=0 0 0.1 rpy=0 0 0
